File: frontpanel/frontpanel.kicad_pcb (KiCad board)
At the start: 2 copper layers, 20 x 128.5 mm, 2 parts

Commit message: :sparkles: Add peace-love-music to frontpanel
Other:
- board text added: "Peace. Love. Music."

Commit message: :fire: Remove parts that should not be visible on the front
Parts:
- removed REF**: OSHW-Logo2_14.6x12mm_SilkScreen, Symbol:OSHW-Logo2_14.6x12mm_SilkScreen
Other:
- board text added: "Peace Love Music"
- board text removed: "CC BY-SA 4.0 Stefan Haun"
- board text removed: "Peace. Love. Music."
- board text removed: "https://github.com/moPsy-project/mousquetaire"
- board text removed: "v1.0"

Commit message: :sparkles: Add design for both module variants
Parts:
- added Ref**: Val**, moPsy_KiCad:moPsy_logo_kicad_20x09_FSilk, B.Cu at (140.0, 157.5)
- moved Ref** 3.37 mm to (140.0, 157.5)
Other:
- outline, holes or cut-outs redrawn
- board text added: "all4one"
- board text added: "one4all"
- board text removed: "Peace Love Music"
